File: Design/H08R7.brd (EAGLE design)
At the start: 34.6 x 30 mm, 26 parts, among them P1 HEXABIT_17.32, U1 STM32G0B1CEU6N, U2 VL53L1CXV0FY_1, X1 XTALL_CSTCE8M00G52

Commit message: -Add TVS diode -Change the MCU to STM32G0B1CEU6 -Activate the thermal option for the polygon - fix the bom
Parts:
- removed C3: 100nF, HEXABITZ_RCLS:C-0603
- removed C4: 4.7uF, HEXABITZ_RCLS:C-0805-POL
- U1: value STM32G0B1CEU6N -> STM32G0B1CEU6QFN_B1CEU6_STM-L; device HEXABITZ_ICs:HEXABITZ_ICS_QFN_B1CEU6_STM-L -> HEXABITZ_ICs:QFN_B1CEU6_STM-L
- moved D2 16.9 mm to (87.9, 64.5), turned to 0 degrees
- moved TRIMBLE-LOGO1 0.67 mm to (74.3, 51.9)
Connections:
- net GND: no longer C3.2, C4.2, U1.30
- net VDD: no longer C3.1, C4.1, U1.31
Routing:
- net GND: track 33.4 -> 55.2 mm, vias 14 -> 13
- net VDD: track 10.1 -> 28.6 mm, vias 2 -> 1
- net USART1_RX: track 16.2 -> 13.9 mm
